File: Bluetooth Multimeter/Bluetooth Multimeter.kicad_sch (KiCad schematic)
At the start: 34 parts, among them J1 V/Ohm, J2 Com, J3 mA, J4 A, J6 3.3V, J7 GND, K1 Low Range, K2 Medium Range, K3 High Range, K4 Ohm Gnd, K5 V/Ohm Switch, U1 ItsyBitsy_NRF52840_Big

Commit message: finalized (fingers crossed) PCB and Schematic
Other:
- company: (none) -> Jayhawk Engineering
- title: (none) -> Bluetooth Multimeter
- moved on the sheet: D1, D10, D11, D2, D3, D4, D5, D6, D7, D8, D9, DS1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
